File: test_project.kicad_sch (KiCad schematic)
At the start: 6 parts, among them U2 TLV62569DBV

Commit message: little changes in schematic and layout
Connections:
- net EN renamed Vin
Other:
- moved on the sheet: C1, C2
Changed lines of the file:
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@@
     (company "Regnum Technology")
-  )
-  (junction (at 109.22 49.53) (diameter 0) (color 0 0 0 0)
-  )
-  (junction (at 163.83 49.53) (diameter 0) (color 0 0 0 0)
-  )
-  (junction (at 109.22 52.07) (diameter 0) (color 0 0 0 0)
   )
   (junction (at 152.4 59.69) (diameter 0) (color 0 0 0 0)
   )
-  (junction (at 109.22 69.85) (diameter 0) (color 0 0 0 0)
+  (junction (at 152.4 49.53) (diameter 0) (color 0 0 0 0)
   )
-  (junction (at 152.4 49.53) (diameter 0) (color 0 0 0 0)
+  (junction (at 114.3 52.07) (diameter 0) (color 0 0 0 0)
   )
   (junction (at 129.54 69.85) (diameter 0) (color 0 0 0 0)
@@
   (junction (at 152.4 69.85) (diameter 0) (color 0 0 0 0)
   )
-  (wire (pts (xy 109.22 60.96) (xy 109.22 69.85))
+  (junction (at 114.3 69.85) (diameter 0) (color 0 0 0 0)
+  )
+  (wire (pts (xy 114.3 60.96) (xy 114.3 69.85))
     (stroke (width 0) (type default))
   )
@@
     (stroke (width 0) (type default))
   )
-  (wire (pts (xy 109.22 69.85) (xy 129.54 69.85))
+  (wire (pts (xy 114.3 52.07) (xy 114.3 53.34))
     (stroke (width 0) (type default))
   )
-  (wire (pts (xy 109.22 52.07) (xy 109.22 53.34))
-    (stroke (width 0) (type default))
-  )
-  (wire (pts (xy 163.83 49.53) (xy 167.64 49.53))
-    (stroke (width 0) (type default))
-  )
-  (wire (pts (xy 104.14 49.53) (xy 109.22 49.53))
-    (stroke (width 0) (type default))
-  )
-  (wire (pts (xy 163.83 69.85) (xy 163.83 63.5))
+  (wire (pts (xy 161.29 69.85) (xy 161.29 63.5))
     (stroke (width 0) (type default))
   )
   (wire (pts (xy 137.16 49.53) (xy 142.24 49.53))
+    (stroke (width 0) (type default))
+  )
+  (wire (pts (xy 114.3 52.07) (xy 121.92 52.07))
+    (stroke (width 0) (type default))
+  )
+  (wire (pts (xy 114.3 69.85) (xy 129.54 69.85))
     (stroke (width 0) (type default))
   )
@@
     (stroke (width 0) (type default))
   )
-  (wire (pts (xy 109.22 49.53) (xy 109.22 52.07))
+  (wire (pts (xy 114.3 49.53) (xy 114.3 52.07))
     (stroke (width 0) (type default))
   )
-  (wire (pts (xy 163.83 49.53) (xy 163.83 55.88))
-    (stroke (width 0) (type default))
-  )
-  (wire (pts (xy 109.22 52.07) (xy 121.92 52.07))
+  (wire (pts (xy 161.29 49.53) (xy 161.29 55.88))
     (stroke (width 0) (type default))
   )
@@
     (stroke (width 0) (type default))
   )
-  (wire (pts (xy 152.4 49.53) (xy 163.83 49.53))
+  (wire (pts (xy 152.4 49.53) (xy 161.29 49.53))
     (stroke (width 0) (type default))
   )
@@
     (stroke (width 0) (type default))
   )
-  (wire (pts (xy 121.92 49.53) (xy 109.22 49.53))
+  (wire (pts (xy 121.92 49.53) (xy 114.3 49.53))
     (stroke (width 0) (type default))
   )
@@
     (stroke (width 0) (type default))
   )
-  (wire (pts (xy 152.4 69.85) (xy 163.83 69.85))
+  (wire (pts (xy 152.4 69.85) (xy 161.29 69.85))
     (stroke (width 0) (type default))
   )
@@
     (effects (font (size 1.27 1.27)) (justify left bottom))
   )
-  (label "EN" (at 119.38 52.07 0) (fields_autoplaced)
-    (effects (font (size 1.27 1.27)) (justify left bottom))
-  )
-  (label "Vin" (at 104.14 49.53 0) (fields_autoplaced)
-    (effects (font (size 1.27 1.27)) (justify left bottom))
+  (label "Vin" (at 114.3 49.53 180) (fields_autoplaced)
+    (effects (font (size 1.27 1.27)) (justify right bottom))
   )
   (label "SW" (at 137.16 49.53 0) (fields_autoplaced)
     (effects (font (size 1.27 1.27)) (justify left bottom))
   )
-  (label "Vout" (at 167.64 49.53 0) (fields_autoplaced)
+  (label "Vout" (at 161.29 49.53 0) (fields_autoplaced)
     (effects (font (size 1.27 1.27)) (justify left bottom))
   )
-  (label "Vin" (at 118.11 49.53 0) (fields_autoplaced)
-    (effects (font (size 1.27 1.27)) (justify left bottom))
-  )
-  (symbol (lib_id "Device:C") (at 109.22 57.15 0) (unit 1)
+  (symbol (lib_id "Device:C") (at 114.3 57.15 0) (unit 1)
     (in_bom yes) (on_board yes) (dnp no)
-    (property "Reference" "C1" (at 110.49 54.61 0)
+    (property "Reference" "C1" (at 115.57 54.61 0)
       (effects (font (size 1.27 1.27)) (justify left))
     )
-    (property "Value" "4.7u" (at 110.49 59.69 0)
+    (property "Value" "4.7u" (at 115.57 59.69 0)
       (effects (font (size 1.27 1.27)) (justify left))
     )
-    (property "Footprint" "Capacitor_SMD:C_0402_1005Metric" (at 110.1852 60.96 0)
+    (property "Footprint" "Capacitor_SMD:C_0402_1005Metric" (at 115.2652 60.96 0)
       (effects (font (size 1.27 1.27)) hide)
     )
-    (property "Datasheet" "~" (at 109.22 57.15 0)
+    (property "Datasheet" "~" (at 114.3 57.15 0)
       (effects (font (size 1.27 1.27)) hide)
     )
@@
     )
   )
-  (symbol (lib_id "Device:C") (at 163.83 59.69 0) (unit 1)
+  (symbol (lib_id "Device:C") (at 161.29 59.69 0) (unit 1)
     (in_bom yes) (on_board yes) (dnp no)
-    (property "Reference" "C2" (at 165.1 57.15 0)
+    (property "Reference" "C2" (at 162.56 57.15 0)
       (effects (font (size 1.27 1.27)) (justify left))
     )
-    (property "Value" "10u" (at 165.1 62.23 0)
+    (property "Value" "10u" (at 162.56 62.23 0)
       (effects (font (size 1.27 1.27)) (justify left))
     )
-    (property "Footprint" "Capacitor_SMD:C_0402_1005Metric" (at 164.7952 63.5 0)
+    (property "Footprint" "Capacitor_SMD:C_0402_1005Metric" (at 162.2552 63.5 0)
       (effects (font (size 1.27 1.27)) hide)
     )
-    (property "Datasheet" "~" (at 163.83 59.69 0)
+    (property "Datasheet" "~" (at 161.29 59.69 0)
       (effects (font (size 1.27 1.27)) hide)
     )
@@
     )
   )
-  (symbol (lib_id "power:GND") (at 109.22 69.85 0) (unit 1)
+  (symbol (lib_id "power:GND") (at 114.3 69.85 0) (unit 1)
     (in_bom yes) (on_board yes) (dnp no) (fields_autoplaced)
-    (property "Reference" "#PWR01" (at 109.22 76.2 0)
+    (property "Reference" "#PWR01" (at 114.3 76.2 0)
       (effects (font (size 1.27 1.27)) hide)
     )
-    (property "Value" "GND" (at 109.22 74.93 0)
+    (property "Value" "GND" (at 114.3 74.93 0)
       (effects (font (size 1.27 1.27)))
     )
-    (property "Footprint" "" (at 109.22 69.85 0)
+    (property "Footprint" "" (at 114.3 69.85 0)
       (effects (font (size 1.27 1.27)) hide)
     )
-    (property "Datasheet" "" (at 109.22 69.85 0)
+    (property "Datasheet" "" (at 114.3 69.85 0)
       (effects (font (size 1.27 1.27)) hide)
     )
