File: test_project.kicad_pcb (KiCad board)
At the start: 2 copper layers, 6 parts, among them U2 TLV62569DBV

Commit message: little changes in schematic and layout
Parts:
- moved C1 0.51 mm to (59.2, 29.0)
Connections:
- net /EN renamed /Vin
Changed lines of the file:
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@@
   (net 1 "GND")
   (net 2 "/Vout")
-  (net 3 "/EN")
+  (net 3 "/Vin")
   (net 4 "/SW")
   (net 5 "/FB")
@@
   )
   (footprint "Capacitor_SMD:C_0402_1005Metric" (layer "F.Cu")
-    (at 58.674 28.956 -90)
+    (at 59.182 28.956 -90)
     (descr "Capacitor SMD 0402 (1005 Metric), square (rectangular) end terminal, IPC_7351 nominal, (Body size source: IPC-SM-782 page 76, https://www.pcb-3d.com/wordpress/wp-content/uploads/ipc-sm-782a_amendment_1_and_2.pdf), generated with kicad-footprint-generator")
     (tags "capacitor")
@@
       (stroke (width 0.1) (type solid)) (layer "F.Fab"))
     (pad "1" smd roundrect (at -0.48 0 270) (size 0.56 0.62) (layers "F.Cu" "F.Paste" "F.Mask") (roundrect_rratio 0.25)
-      (net 3 "/EN") (pintype "passive"))
+      (net 3 "/Vin") (pintype "passive"))
     (pad "2" smd roundrect (at 0.48 0 270) (size 0.56 0.62) (layers "F.Cu" "F.Paste" "F.Mask") (roundrect_rratio 0.25)
       (net 1 "GND") (pintype "passive"))
@@
       (stroke (width 0.1) (type solid)) (layer "F.Fab"))
     (pad "1" smd roundrect (at -1.1375 -0.95 180) (size 1.325 0.6) (layers "F.Cu" "F.Paste" "F.Mask") (roundrect_rratio 0.25)
-      (net 3 "/EN") (pinfunction "EN") (pintype "input"))
+      (net 3 "/Vin") (pinfunction "EN") (pintype "input"))
     (pad "2" smd roundrect (at -1.1375 0 180) (size 1.325 0.6) (layers "F.Cu" "F.Paste" "F.Mask") (roundrect_rratio 0.25)
       (net 1 "GND") (pinfunction "GND") (pintype "power_in"))
@@
       (net 4 "/SW") (pinfunction "SW") (pintype "power_out"))
     (pad "4" smd roundrect (at 1.1375 0.95 180) (size 1.325 0.6) (layers "F.Cu" "F.Paste" "F.Mask") (roundrect_rratio 0.25)
-      (net 3 "/EN") (pinfunction "VIN") (pintype "power_in"))
+      (net 3 "/Vin") (pinfunction "VIN") (pintype "power_in"))
     (pad "5" smd roundrect (at 1.1375 -0.95 180) (size 1.325 0.6) (layers "F.Cu" "F.Paste" "F.Mask") (roundrect_rratio 0.25)
       (net 5 "/FB") (pinfunction "FB") (pintype "input"))
@@
     (connect_pads yes (clearance 0.5))
     (min_thickness 0.25) (filled_areas_thickness no)
-    (fill yes (thermal_gap 0.5) (thermal_bridge_width 0.5))
+    (fill (thermal_gap 0.5) (thermal_bridge_width 0.5))
     (polygon
       (pts
-        (xy 70.104 29.21)
+        (xy 71.374 29.21)
         (xy 56.896 29.21)
         (xy 56.896 36.068)
-        (xy 70.104 36.068)
+        (xy 71.374 36.068)
       )
     )
   )
-  (zone (net 3) (net_name "/EN") (layer "F.Cu") (hatch edge 0.5)
+  (zone (net 3) (net_name "/Vin") (layer "F.Cu") (hatch edge 0.5)
     (priority 2)
     (connect_pads yes (clearance 0.5))
     (min_thickness 0.25) (filled_areas_thickness no)
-    (fill yes (thermal_gap 0.5) (thermal_bridge_width 0.5))
+    (fill (thermal_gap 0.5) (thermal_bridge_width 0.5))
     (polygon
       (pts
         (xy 61.722 28.956)
         (xy 56.896 28.956)
-        (xy 56.896 22.606)
-        (xy 59.436 22.606)
-        (xy 59.436 27.94)
+        (xy 56.896 21.336)
+        (xy 60.198 21.336)
+        (xy 60.198 26.924)
+        (xy 60.96 27.94)
         (xy 61.722 27.94)
       )
@@
     (connect_pads yes (clearance 0.5))
     (min_thickness 0.25) (filled_areas_thickness no)
-    (fill yes (thermal_gap 0.5) (thermal_bridge_width 0.5))
+    (fill (thermal_gap 0.5) (thermal_bridge_width 0.5))
     (polygon
       (pts
         (xy 65.532 22.606)
         (xy 65.532 28.956)
-        (xy 70.104 28.956)
-        (xy 70.104 22.606)
-        (xy 69.088 22.606)
-        (xy 67.818 25.654)
+        (xy 71.374 28.956)
+        (xy 71.374 21.336)
+        (xy 68.58 21.336)
+        (xy 68.072 24.892)
+        (xy 67.818 24.892)
         (xy 67.818 22.606)
       )

Commit message: pcb edited
Parts:
- moved C1 106.0 mm to (140.5, 97.0)
- moved C2 106.0 mm to (147.6, 97.0)
- moved U2 106.0 mm to (143.4, 97.5)
- moved L1 106.0 mm to (145.8, 92.1)
- moved R2 104.8 mm to (142.7, 100.3)
- moved R1 104.7 mm to (142.8, 101.9)
Routing:
- net /Vin: track 0.00 -> 3.07 mm
- net /Vout: track 11.7 -> 11.0 mm
Other:
- board outline added: 15 x 15.5 mm
Changed lines of the file:
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@@
   )
   (paper "A4")
+  (title_block
+    (title "buck converter pcb")
+    (date "2023-09-06")
+  )
   (layers
     (0 "F.Cu" signal)
@@
     )
     (pad_to_mask_clearance 0)
+    (grid_origin 135.636 106.934)
     (pcbplotparams
       (layerselection 0x00010fc_ffffffff)
@@
   (net 5 "/FB")
   (footprint "Resistor_SMD:R_0402_1005Metric" (layer "F.Cu")
-    (at 61.974 33.528)
+    (at 142.748 100.33)
     (descr "Resistor SMD 0402 (1005 Metric), square (rectangular) end terminal, IPC_7351 nominal, (Body size source: IPC-SM-782 page 72, https://www.pcb-3d.com/wordpress/wp-content/uploads/ipc-sm-782a_amendment_1_and_2.pdf), generated with kicad-footprint-generator")
     (tags "resistor")
@@
   )
   (footprint "Inductor_SMD:L_Chilisin_BMRB00050518-B" (layer "F.Cu")
-    (at 64.516 24.13 180)
+    (at 145.807 92.136 180)
     (descr "Inductor, Chilisin, BMRB00050518-B, 5.4x5.2x1.6mm, https://www.chilisin.com/upload/media/product/power/file/BMRx_Series.pdf")
     (tags "Inductor bmrx mchi")
@@
   )
   (footprint "Capacitor_SMD:C_0402_1005Metric" (layer "F.Cu")
-    (at 59.182 28.956 -90)
+    (at 140.473 96.962 -90)
     (descr "Capacitor SMD 0402 (1005 Metric), square (rectangular) end terminal, IPC_7351 nominal, (Body size source: IPC-SM-782 page 76, https://www.pcb-3d.com/wordpress/wp-content/uploads/ipc-sm-782a_amendment_1_and_2.pdf), generated with kicad-footprint-generator")
     (tags "capacitor")
@@
   )
   (footprint "Package_TO_SOT_SMD:SOT-23-5" (layer "F.Cu")
-    (at 62.0975 29.53 180)
+    (at 143.3885 97.536 180)
     (descr "SOT, 5 Pin (https://www.jedec.org/sites/default/files/docs/Mo-178c.PDF variant AA), generated with kicad-footprint-generator ipc_gullwing_generator.py")
     (tags "SOT TO_SOT_SMD")
@@
   )
   (footprint "Resistor_SMD:R_0402_1005Metric" (layer "F.Cu")
-    (at 61.976 35.306 180)
+    (at 142.759 101.854 180)
     (descr "Resistor SMD 0402 (1005 Metric), square (rectangular) end terminal, IPC_7351 nominal, (Body size source: IPC-SM-782 page 72, https://www.pcb-3d.com/wordpress/wp-content/uploads/ipc-sm-782a_amendment_1_and_2.pdf), generated with kicad-footprint-generator")
     (tags "resistor")
@@
   )
   (footprint "Capacitor_SMD:C_0402_1005Metric" (layer "F.Cu")
-    (at 66.294 28.984 -90)
+    (at 147.585 96.99 -90)
     (descr "Capacitor SMD 0402 (1005 Metric), square (rectangular) end terminal, IPC_7351 nominal, (Body size source: IPC-SM-782 page 76, https://www.pcb-3d.com/wordpress/wp-content/uploads/ipc-sm-782a_amendment_1_and_2.pdf), generated with kicad-footprint-generator")
     (tags "capacitor")
@@
     )
   )
-  (segment (start 62.486 35.306) (end 64.262 35.306) (width 0.25) (layer "F.Cu") (net 2))
-  (via (at 67.818 28.194) (size 0.8) (drill 0.4) (layers "F.Cu" "B.Cu") (net 2))
-  (via (at 64.262 35.306) (size 0.8) (drill 0.4) (layers "F.Cu" "B.Cu") (net 2))
-  (segment (start 67.818 34.036) (end 66.548 35.306) (width 0.25) (layer "B.Cu") (net 2))
-  (segment (start 67.818 28.194) (end 67.818 34.036) (width 0.25) (layer "B.Cu") (net 2))
-  (segment (start 66.548 35.306) (end 64.262 35.306) (width 0.25) (layer "B.Cu") (net 2))
-  (segment (start 61.466 33.528) (end 60.96 33.022) (width 0.25) (layer "F.Cu") (net 5))
-  (segment (start 60.96 33.022) (end 60.96 30.48) (width 0.25) (layer "F.Cu") (net 5))
+  (gr_rect (start 137.922 87.884) (end 152.908 103.378)
+    (stroke (width 0.1) (type default)) (fill none) (layer "Edge.Cuts"))
+  (segment (start 143.269 101.854) (end 145.542 101.854) (width 0.25) (layer "F.Cu") (net 2))
+  (via (at 149.109 96.2) (size 0.8) (drill 0.4) (layers "F.Cu" "B.Cu") (net 2))
+  (via (at 145.542 101.854) (size 0.8) (drill 0.4) (layers "F.Cu" "B.Cu") (net 2))
+  (segment (start 145.542 101.854) (end 148.336 101.854) (width 0.25) (layer "B.Cu") (net 2))
+  (segment (start 149.109 101.081) (end 149.109 96.2) (width 0.25) (layer "B.Cu") (net 2))
+  (segment (start 148.336 101.854) (end 149.109 101.081) (width 0.25) (layer "B.Cu") (net 2))
+  (segment (start 142.251 96.595251) (end 142.251 96.586) (width 0.25) (layer "F.Cu") (net 3))
+  (segment (start 144.526 98.486) (end 144.141749 98.486) (width 0.25) (layer "F.Cu") (net 3))
+  (segment (start 144.141749 98.486) (end 142.251 96.595251) (width 0.25) (layer "F.Cu") (net 3))
+  (segment (start 142.24 101.845) (end 142.249 101.854) (width 0.25) (layer "F.Cu") (net 5))
+  (segment (start 142.251 98.541) (end 142.24 98.552) (width 0.25) (layer "F.Cu") (net 5))
+  (segment (start 142.24 98.552) (end 142.24 101.845) (width 0.25) (layer "F.Cu") (net 5))
+  (segment (start 142.251 98.486) (end 142.251 98.541) (width 0.25) (layer "F.Cu") (net 5))
   (zone (net 1) (net_name "GND") (layer "F.Cu") (hatch edge 0.5)
     (connect_pads yes (clearance 0.5))
     (min_thickness 0.25) (filled_areas_thickness no)
-    (fill (thermal_gap 0.5) (thermal_bridge_width 0.5))
+    (fill yes (thermal_gap 0.5) (thermal_bridge_width 0.5))
     (polygon
       (pts
-        (xy 71.374 29.21)
-        (xy 56.896 29.21)
-        (xy 56.896 36.068)
-        (xy 71.374 36.068)
+        (xy 152.665 97.216)
+        (xy 138.187 97.216)
+        (xy 138.187 103.312)
+        (xy 152.665 103.312)
       )
     )
   )
-  (zone (net 3) (net_name "/Vin") (layer "F.Cu") (hatch edge 0.5)
+  (zone (net 3) (net_name "/Vin") (layer "F.Cu") (hatch edge 0.508)
     (priority 2)
-    (connect_pads yes (clearance 0.5))
-    (min_thickness 0.25) (filled_areas_thickness no)
-    (fill (thermal_gap 0.5) (thermal_bridge_width 0.5))
+    (connect_pads yes (clearance 0.508))
+    (min_thickness 0.254) (filled_areas_thickness no)
+    (fill yes (thermal_gap 0.508) (thermal_bridge_width 0.508))
     (polygon
       (pts
-        (xy 61.722 28.956)
-        (xy 56.896 28.956)
-        (xy 56.896 21.336)
-        (xy 60.198 21.336)
-        (xy 60.198 26.924)
-        (xy 60.96 27.94)
-        (xy 61.722 27.94)
+        (xy 143.013 96.962)
+        (xy 138.187 96.962)
+        (xy 138.187 89.342)
+        (xy 141.997 89.342)
+        (xy 141.997 94.996)
+        (xy 142.494 95.504)
+        (xy 143.002 96.012)
       )
     )
@@
     (connect_pads yes (clearance 0.5))
     (min_thickness 0.25) (filled_areas_thickness no)
-    (fill (thermal_gap 0.5) (thermal_bridge_width 0.5))
+    (fill yes (thermal_gap 0.5) (thermal_bridge_width 0.5))
     (polygon
       (pts
-        (xy 65.532 22.606)
-        (xy 65.532 28.956)
-        (xy 71.374 28.956)
-        (xy 71.374 21.336)
-        (xy 68.58 21.336)
-        (xy 68.072 24.892)
-        (xy 67.818 24.892)
-        (xy 67.818 22.606)
+        (xy 146.823 90.612)
+        (xy 146.823 96.962)
+        (xy 152.665 96.962)
+        (xy 152.665 89.342)
+        (xy 149.871 89.342)
+        (xy 149.86 93.726)
+        (xy 149.109 93.726)
+        (xy 149.109 90.612)
       )
     )
@@
     (polygon
       (pts
-        (xy 64.008 28.956)
-        (xy 64.008 27.94)
-        (xy 63.754 27.432)
-        (xy 63.754 22.606)
-        (xy 61.214 22.606)
-        (xy 61.214 27.432)
-        (xy 62.484 27.94)
-        (xy 62.484 28.956)
+        (xy 145.299 96.962)
+        (xy 145.299 95.946)
+        (xy 145.299 95.438)
+        (xy 145.299 90.612)
+        (xy 142.505 90.612)
+        (xy 142.494 94.742)
+        (xy 143.764 96.012)
+        (xy 143.775 96.962)
       )
     )
